File: PD_ElectrodeBoard_v4/PD_ElectrodeBoard_v4.sch (KiCad schematic (older format))
At the start: 123 parts, among them J1 Conn_02x32_Odd_Even, J10 Conn_01x02, J11 TopPlate, J2 Conn_02x32_Odd_Even, J3 Conn_01x02, J4 Conn_01x02, J5 Conn_01x02, J6 Conn_01x02, J7 Conn_01x02, J8 Conn_01x02, J9 Conn_01x02, T1 ZNI1000, T2 ZNI1000, T3 ZNI1000, T4 ZNI1000

Commit message: new revision 4.1 of electrode board
Parts:
- removed E201, E202, E203: ReservoirB, electrodes:reservoir_B_2.50mm, symbol Electrodes:ReservoirB
- removed J10, J3, J4, J5, J6, J7, J8, J9: Conn_01x02, PurpleDrop:SMT_PADS_1x2, symbol Connector_Generic:Conn_01x02
- removed R5: 0, Resistor_SMD:R_0603_1608Metric_Pad1.05x0.95mm_HandSolder, symbol Device:R_US
- added E201, E202, E203: Reservoir, electrodes:reservoir_A_2.25mm, symbol Electrodes:Reservoir
- added E96, E97, E98: DMFElectrode, electrodes:electrode_points_1_40deg_trbl, symbol Electrodes:DMFElectrode
- added G1: AprilTag, PurpleDrop:tag36_11_00004_6.00mm, symbol PurpleDrop:AprilTag
- added G2: AprilTag, PurpleDrop:tag36_11_00005_6.00mm, symbol PurpleDrop:AprilTag
- added G3: AprilTag, PurpleDrop:tag36_11_00006_6.00mm, symbol PurpleDrop:AprilTag
- added J3: HEAT, Connector_JST:JST_PH_S5B-PH-SM4-TB_1x05-1MP_P2.00mm_Horizontal, symbol Connector_Generic:Conn_01x05
- added J4: RTD, Connector_JST:JST_PH_S8B-PH-SM4-TB_1x08-1MP_P2.00mm_Horizontal, symbol Connector_Generic:Conn_01x08
- E1, E10, E11, E12, E13, E14, E15, E16, E17, E18, E19, E2, E20, E21, E22, E23, E24, E25, E26, E27, E28, E29, E3, E30, E31, E32, E33, E34, E35, E36, E37, E38, E39, E4, E40, E41, E42, E43, E44, E45, E46, E47, E48, E49, E5, E50, E51, E52, E53, E54, E55, E56, E57, E58, E59, E6, E60, E61, E62, E63, E64, E65, E66, E67, E68, E69, E7, E70, E71, E72, E73, E74, E75, E76, E77, E78, E79, E8, E80, E81, E82, E83, E84, E85, E86, E87, E88, E89, E9, E90, E91, E92, E93, E94, E95: footprint electrodes:electrode_points_2_45deg -> electrodes:electrode_points_1_40deg_trbl
- E200: footprint electrodes:reservoir_A_2.50mm -> electrodes:reservoir_A_2.25mm
- H1, H2, H3, H4: footprint PurpleDrop:NPTH3.7 -> PurpleDrop:Keystone-4929
- R1, R2, R3, R4: footprint Package_TO_SOT_SMD:TO-252-2 -> PurpleDrop:PWR163_Resistor_DPAK
Connections:
- net P0: now also E52.1, J2.34 (Pin_34); no longer E44.1, J2.32 (Pin_32)
- net P1: now also E41.1, J2.36 (Pin_36); no longer E45.1, J2.30 (Pin_30)
- net P10: now also E13.1, J2.54 (Pin_54); no longer E71.1, J2.12 (Pin_12)
- net P100: now also E56.1, J1.42 (Pin_42); no longer J1.24 (Pin_24)
- net P101: now also E57.1, J1.44 (Pin_44); no longer E90.1, J1.22 (Pin_22), R4.2 (TAB), T4.3 (PROBE)
- net P102: now also E46.1, J1.46 (Pin_46); no longer E88.1, J1.20 (Pin_20), R2.2 (TAB), T2.3 (PROBE)
- net P103: now also E47.1, J1.48 (Pin_48); no longer E86.1, J1.18 (Pin_18)
- net P104: now also E36.1, J1.50 (Pin_50); no longer E78.1, J1.16 (Pin_16)
- net P105: now also E37.1, J1.52 (Pin_52); no longer E79.1, J1.14 (Pin_14)
- net P106: now also E27.1, J1.54 (Pin_54); no longer E80.1, J1.12 (Pin_12)
- net P107: now also E26.1, J1.56 (Pin_56); no longer E81.1, J1.10 (Pin_10)
- net P108: now also E17.1, J1.58 (Pin_58); no longer E82.1, J1.8 (Pin_8)
- net P109: now also E16.1, J1.60 (Pin_60); no longer E65.1, J1.6 (Pin_6)
- net P11: now also E3.1, J2.56 (Pin_56); no longer J2.10 (Pin_10)
- net P110: now also E7.1, J1.62 (Pin_62); no longer E66.1, J1.4 (Pin_4)
- net P111: now also E6.1, J1.64 (Pin_64); no longer E83.1, J1.2 (Pin_2)
- net P112: now also E9.1, J1.63 (Pin_63); no longer E67.1, J1.1 (Pin_1)
- net P113: now also E10.1, J1.61 (Pin_61); no longer E84.1, J1.3 (Pin_3)
- net P114: now also J1.59 (Pin_59), E202.1; no longer E68.1, J1.5 (Pin_5)
- net P115: now also E19.1, J1.57 (Pin_57); no longer E69.1, J1.7 (Pin_7)
- net P116: now also J1.55 (Pin_55), E202.2; no longer E70.1, J1.9 (Pin_9)
- net P117: now also E20.1, J1.53 (Pin_53); no longer J1.11 (Pin_11)
- net P118: now also E29.1, J1.51 (Pin_51); no longer J1.13 (Pin_13)
- net P119: now also E30.1, J1.49 (Pin_49); no longer J1.15 (Pin_15)
- net P12: now also E200.2, J2.58 (Pin_58); no longer E61.1, J2.8 (Pin_8)
- net P120: now also E39.1, J1.47 (Pin_47); no longer J1.17 (Pin_17)
- net P121: now also E40.1, J1.45 (Pin_45); no longer J1.19 (Pin_19)
- net P122: now also E49.1, J1.43 (Pin_43); no longer E64.1, J1.21 (Pin_21)
- net P123: now also J1.41 (Pin_41); no longer J1.23 (Pin_23)
- net P124: now also E59.1, J1.39 (Pin_39); no longer E54.1, J1.25 (Pin_25)
- net P125: now also E60.1, J1.37 (Pin_37); no longer E55.1, J1.27 (Pin_27)
- net P126: now also E69.1, J1.35 (Pin_35); no longer E56.1, J1.29 (Pin_29)
- net P127: now also E70.1, J1.33 (Pin_33); no longer E53.1, J1.31 (Pin_31)
- net P13: now also E200.1, J2.60 (Pin_60); no longer E72.1, J2.6 (Pin_6)
- net P14: now also E1.1, J2.62 (Pin_62); no longer E60.1, J2.4 (Pin_4)
- net P15: now also E2.1, J2.64 (Pin_64); no longer E62.1, J2.2 (Pin_2)
- net P16: now also E4.1, J2.63 (Pin_63); no longer E73.1, J2.1 (Pin_1)
- net P17: now also E5.1, J2.61 (Pin_61); no longer E49.1, J2.3 (Pin_3)
- net P18: now also E15.1, J2.59 (Pin_59); no longer E74.1, J2.5 (Pin_5)
- net P19: now also E14.1, J2.57 (Pin_57); no longer E63.1, J2.7 (Pin_7)
- net P2: now also E42.1, J2.38 (Pin_38); no longer E58.1, J2.28 (Pin_28)
- net P20: now also E25.1, J2.55 (Pin_55); no longer E77.1, J2.9 (Pin_9)
- net P21: now also E24.1, J2.53 (Pin_53); no longer E75.1, J2.11 (Pin_11)
- net P22: now also E35.1, J2.51 (Pin_51); no longer E76.1, J2.13 (Pin_13)
- net P23: now also E23.1, J2.49 (Pin_49); no longer E85.1, J2.15 (Pin_15)
- net P24: now also E34.1, J2.47 (Pin_47); no longer E87.1, J2.17 (Pin_17), R1.2 (TAB), T1.3 (PROBE)
- net P25: now also E45.1, J2.45 (Pin_45); no longer E89.1, J2.19 (Pin_19), R3.2 (TAB), T3.3 (PROBE)
- net P26: now also E44.1, J2.43 (Pin_43); no longer J2.21 (Pin_21)
- net P27: now also E55.1, J2.41 (Pin_41); no longer J2.23 (Pin_23)
- net P28: now also E54.1, J2.39 (Pin_39); no longer J2.25 (Pin_25)
- net P29: now also E65.1, J2.37 (Pin_37); no longer J2.27 (Pin_27)
- net P3: now also E31.1, J2.40 (Pin_40); no longer E57.1, J2.26 (Pin_26)
- net P30: now also E64.1, J2.35 (Pin_35); no longer J2.29 (Pin_29)
- net P31: now also E75.1, J2.33 (Pin_33); no longer J2.31 (Pin_31)
- net P32: now also E74.1, J2.31 (Pin_31); no longer J2.33 (Pin_33)
- net P33: now also E85.1, J2.29 (Pin_29); no longer J2.35 (Pin_35)
- net P34: now also E84.1, J2.27 (Pin_27); no longer J2.37 (Pin_37)
- net P35: now also E43.1, J2.25 (Pin_25); no longer E91.1, J2.39 (Pin_39)
- net P36: now also E53.1, J2.23 (Pin_23); no longer E93.1, J2.41 (Pin_41)
- net P37: now also E63.1, J2.21 (Pin_21); no longer E7.1, J2.43 (Pin_43)
- net P38: now also E73.1, J2.19 (Pin_19); no longer E21.1, J2.45 (Pin_45)
- net P39: now also E83.1, J2.17 (Pin_17); no longer E35.1, J2.47 (Pin_47)
- net P4: now also E32.1, J2.42 (Pin_42); no longer J2.24 (Pin_24)
- net P40: now also E91.1, J2.15 (Pin_15); no longer E6.1, J2.49 (Pin_49)
- net P41: now also E93.1, J2.13 (Pin_13); no longer E20.1, J2.51 (Pin_51)
- net P42: now also J2.11 (Pin_11); no longer E34.1, J2.53 (Pin_53)
- net P43: now also J2.9 (Pin_9); no longer E5.1, J2.55 (Pin_55)
- net P44: now also J2.7 (Pin_7); no longer E19.1, J2.57 (Pin_57)
- net P45: now also J2.5 (Pin_5); no longer E4.1, J2.59 (Pin_59)
- net P46: now also J2.3 (Pin_3); no longer E18.1, J2.61 (Pin_61)
- net P47: now also J2.1 (Pin_1); no longer E3.1, J2.63 (Pin_63)
- net P48: now also J2.2 (Pin_2); no longer E17.1, J2.64 (Pin_64)
- net P49: now also J2.4 (Pin_4); no longer E2.1, J2.62 (Pin_62)
- net P5: now also E21.1, J2.44 (Pin_44); no longer J2.22 (Pin_22)
- net P50: now also J2.6 (Pin_6); no longer E16.1, J2.60 (Pin_60)
- net P51: now also J2.8 (Pin_8); no longer E15.1, J2.58 (Pin_58)
- net P52: now also J2.10 (Pin_10); no longer E1.1, J2.56 (Pin_56)
- net P53: now also J2.12 (Pin_12), R3.2 (TAB), T3.3 (PROBE), E97.1; no longer E95.1, J2.54 (Pin_54)
- net P54: now also E95.1, J2.14 (Pin_14), R1.2 (TAB), T1.3 (PROBE); no longer E200.1, J2.52 (Pin_52)
- net P55: now also E81.1, J2.16 (Pin_16); no longer E200.2, J2.50 (Pin_50)
- net P56: now also J2.18 (Pin_18), E201.2; no longer E31.1, J2.48 (Pin_48)
- net P57: now also J2.20 (Pin_20), E201.1; no longer E30.1, J2.46 (Pin_46)
- net P58: now also E82.1, J2.22 (Pin_22); no longer E29.1, J2.44 (Pin_44)
- net P59: now also E71.1, J2.24 (Pin_24); no longer E32.1, J2.42 (Pin_42)
- net P6: now also E22.1, J2.46 (Pin_46); no longer J2.20 (Pin_20)
- net P60: now also E72.1, J2.26 (Pin_26); no longer E33.1, J2.40 (Pin_40)
- net P61: now also E61.1, J2.28 (Pin_28); no longer E47.1, J2.38 (Pin_38)
- net P62: now also E62.1, J2.30 (Pin_30); no longer E46.1, J2.36 (Pin_36)
- net P63: now also E51.1, J2.32 (Pin_32); no longer E43.1, J2.34 (Pin_34)
- net P64: now also E79.1, J1.31 (Pin_31); no longer E52.1, J1.33 (Pin_33)
- net P65: now also E80.1, J1.29 (Pin_29); no longer E38.1, J1.35 (Pin_35)
- net P66: now also E48.1, J1.27 (Pin_27); no longer E39.1, J1.37 (Pin_37)
- net P67: now also E58.1, J1.25 (Pin_25); no longer E42.1, J1.39 (Pin_39)
- net P68: now also J1.23 (Pin_23); no longer E41.1, J1.41 (Pin_41)
- net P69: now also E68.1, J1.21 (Pin_21); no longer E40.1, J1.43 (Pin_43)
- net P7: now also E33.1, J2.48 (Pin_48); no longer J2.18 (Pin_18)
- net P70: now also E78.1, J1.19 (Pin_19); no longer J1.45 (Pin_45)
- net P71: now also E90.1, J1.17 (Pin_17); no longer J1.47 (Pin_47)
- net P72: now also E89.1, J1.15 (Pin_15); no longer J1.49 (Pin_49)
- net P73: now also J1.13 (Pin_13), E203.1; no longer J1.51 (Pin_51)
- net P74: now also E87.1, J1.11 (Pin_11); no longer J1.53 (Pin_53)
- net P75: now also J1.9 (Pin_9), E203.2; no longer E28.1, J1.55 (Pin_55)
- net P76: now also E92.1, J1.7 (Pin_7); no longer E27.1, J1.57 (Pin_57)
- net P77: now also E94.1, J1.5 (Pin_5); no longer E14.1, J1.59 (Pin_59)
- net P78: now also J1.3 (Pin_3), R2.2 (TAB), T2.3 (PROBE), E96.1; no longer E13.1, J1.61 (Pin_61)
- net P79: now also J1.1 (Pin_1), R4.2 (TAB), T4.3 (PROBE), E98.1; no longer E26.1, J1.63 (Pin_63)
- net P8: now also E11.1, J2.50 (Pin_50); no longer E48.1, J2.16 (Pin_16)
- net P80: now also J1.2 (Pin_2); no longer E12.1, J1.64 (Pin_64)
- net P81: now also J1.4 (Pin_4); no longer E25.1, J1.62 (Pin_62)
- net P82: now also E88.1, J1.6 (Pin_6); no longer E11.1, J1.60 (Pin_60)
- net P83: now also E86.1, J1.8 (Pin_8); no longer E37.1, J1.58 (Pin_58)
- net P84: now also J1.10 (Pin_10); no longer E24.1, J1.56 (Pin_56)
- net P85: now also J1.12 (Pin_12); no longer E51.1, J1.54 (Pin_54)
- net P86: now also J1.14 (Pin_14); no longer E10.1, J1.52 (Pin_52)
- net P87: now also J1.16 (Pin_16); no longer E23.1, J1.50 (Pin_50)
- net P88: now also J1.18 (Pin_18); no longer E36.1, J1.48 (Pin_48)
- net P89: now also J1.20 (Pin_20); no longer E9.1, J1.46 (Pin_46)
- net P9: now also E12.1, J2.52 (Pin_52); no longer E59.1, J2.14 (Pin_14)
- net P90: now also E28.1, J1.22 (Pin_22); no longer E22.1, J1.44 (Pin_44)
- net P91: now also E76.1, J1.24 (Pin_24); no longer E8.1, J1.42 (Pin_42)
- net P92: now also E77.1, J1.26 (Pin_26); no longer E94.1, J1.40 (Pin_40)
- net P93: now also E38.1, J1.28 (Pin_28); no longer E92.1, J1.38 (Pin_38)
- net P94: now also J1.30 (Pin_30); no longer J1.36 (Pin_36), J11.1 (Pin_1)
- net P95: now also E18.1, J1.32 (Pin_32); no longer J1.34 (Pin_34)
- net P96: now also E8.1, J1.34 (Pin_34); no longer J1.32 (Pin_32)
- net P97: now also J1.36 (Pin_36), J11.1 (Pin_1); no longer J1.30 (Pin_30)
- net P98: now also E66.1, J1.38 (Pin_38); no longer J1.28 (Pin_28)
- net P99: now also E67.1, J1.40 (Pin_40); no longer J1.26 (Pin_26)
- net at R2.1: now also J3.2 (Pin_2)
- net at R2.3: now also R1.3, R3.3, R4.3, J3.5 (Pin_5)
- net at R3.1: now also J3.3 (Pin_3)
- net at R4.1: now also J3.4 (Pin_4)
- net at R1.1: now also J3.1 (Pin_1)
- net RTD1_A: now reaches T1.1 (R1)
- net RTD1_A: now also J4.1 (Pin_1)
- net RTD1_B: now reaches T1.2 (R2)
- net RTD1_B: now also J4.2 (Pin_2)
- net RTD2_A: now reaches T2.1 (R1)
- net RTD2_A: now also J4.3 (Pin_3)
- net RTD2_B: now reaches T2.2 (R2)
- net RTD2_B: now also J4.4 (Pin_4)
- net RTD3_A: now reaches T3.1 (R1)
- net RTD3_A: now also J4.5 (Pin_5)
- net RTD3_B: now reaches T3.2 (R2)
- net RTD3_B: now also J4.6 (Pin_6)
- net RTD4_A: now reaches T4.1 (R1)
- net RTD4_A: now also J4.7 (Pin_7)
- net RTD4_B: now reaches T4.2 (R2)
- net RTD4_B: now also J4.8 (Pin_8)
- net POUR: now reaches H4.1
- net POUR: now also H1.1, H2.1, H3.1
Other:
- note removed: "Short to connect guard pour around electrodes to top plate voltage"
- moved on the sheet: E85, E86, E87, E88, E89, E90, E91, E92, E93, E94, E95, H1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
